File: hardware/resistor_load/resistor_load.kicad_pcb (KiCad board)
At the start: 2 copper layers, 50 x 50 mm, 7 parts, among them J1 Conn_02x03_Odd_Even, J2 Conn_02x03_Odd_Even

Commit message: added test pads to fixture boards
Parts:
- added TP1: P1+, TestPoint:TestPoint_Pad_1.5x1.5mm, F.Cu at (146.8, 74.7)
- added TP2: P2+, TestPoint:TestPoint_Pad_1.5x1.5mm, F.Cu at (144.1, 82.1)
- added TP3: P3+, TestPoint:TestPoint_Pad_1.5x1.5mm, F.Cu at (143.8, 88.1)
- added TP4: P3-, TestPoint:TestPoint_Pad_1.5x1.5mm, F.Cu at (157.3, 88.9)
- added TP5: P2-, TestPoint:TestPoint_Pad_1.5x1.5mm, F.Cu at (157.6, 82.2)
- added TP6: P1-, TestPoint:TestPoint_Pad_1.5x1.5mm, F.Cu at (157.4, 74.7)
Routing:
- net /P3+: track 11.7 -> 16.9 mm
- net /P2-: track 28.7 -> 33.5 mm
- net /P3-: track 30.6 -> 35.2 mm
- net /P1-: track 33.1 -> 37.6 mm
- net /P1+: track 12.4 -> 16.5 mm
- net /P2+: track 8.83 -> 11.3 mm
Other:
- board text added: "Biobattery Resistive Test Load v1.1 (2026/07/01)"
- board text removed: "Air Battery 47kOhm Resistor Test Load v1.0 (2024/04/17)"
