File: hardware/resistor_load/resistor_load.kicad_sch (KiCad schematic)
At the start: 5 parts, among them J1 Conn_02x03_Odd_Even, J2 Conn_02x03_Odd_Even

Commit message: added test pads to fixture boards
Parts:
- added TP1, TP2, TP3, TP4, TP5, TP6: TestPoint, TestPoint:TestPoint_Pad_1.5x1.5mm, symbol Connector:TestPoint
Connections:
- net P1+: now also TP1.1
- net P1-: now also TP6.1
- net P2+: now also TP2.1
- net P2-: now also TP5.1
- net P3+: now also TP3.1
- net P3-: now also TP4.1
